Commit message: Update urdf files

File: src/assets/revo2/urdf/revo2_right_hand.urdf (robot description, URDF)
Before this commit: robot brainco_revo2_righthand_urdf, 22 links, 21 joints
Links:
- link right_base_link: geometry collision mesh filename=../meshes/right_base_link.obj; visual mesh filename=../meshes/right_base_link.obj
- link right_index_distal_link: geometry collision mesh filename=../meshes/right_index_distal_link.obj; visual mesh filename=../meshes/right_index_distal_link.obj
- link right_index_proximal_link: geometry collision mesh filename=../meshes/right_index_proximal_link.obj; visual mesh filename=../meshes/right_index_proximal_link.obj
- link right_index_touch_link: geometry collision mesh filename=../meshes/right_index_touch_link.obj; visual mesh filename=../meshes/right_index_touch_link.obj
- link right_middle_distal_link: geometry collision mesh filename=../meshes/right_middle_distal_link.obj; visual mesh filename=../meshes/right_middle_distal_link.obj
- link right_middle_proximal_link: geometry collision mesh filename=../meshes/right_middle_proximal_link.obj; visual mesh filename=../meshes/right_middle_proximal_link.obj
- link right_middle_touch_link: geometry collision mesh filename=../meshes/right_middle_touch_link.obj; visual mesh filename=../meshes/right_middle_touch_link.obj
- link right_pinky_distal_link: geometry collision mesh filename=../meshes/right_pinky_distal_link.obj; visual mesh filename=../meshes/right_pinky_distal_link.obj
- link right_pinky_proximal_link: geometry collision mesh filename=../meshes/right_pinky_proximal_link.obj; visual mesh filename=../meshes/right_pinky_proximal_link.obj
- link right_pinky_touch_link: geometry collision mesh filename=../meshes/right_pinky_touch_link.obj; visual mesh filename=../meshes/right_pinky_touch_link.obj
- link right_ring_distal_link: geometry collision mesh filename=../meshes/right_ring_distal_link.obj; visual mesh filename=../meshes/right_ring_distal_link.obj
- link right_ring_proximal_link: geometry collision mesh filename=../meshes/right_ring_proximal_link.obj; visual mesh filename=../meshes/right_ring_proximal_link.obj
- link right_ring_touch_link: geometry collision mesh filename=../meshes/right_ring_touch_link.obj; visual mesh filename=../meshes/right_ring_touch_link.obj
- link right_thumb_distal_link: geometry collision mesh filename=../meshes/right_thumb_distal_link.obj; visual mesh filename=../meshes/right_thumb_distal_link.obj
- link right_thumb_metacarpal_link: geometry collision mesh filename=../meshes/right_thumb_metacarpal_link.obj; visual mesh filename=../meshes/right_thumb_metacarpal_link.obj
- link right_thumb_proximal_link: geometry collision mesh filename=../meshes/right_thumb_proximal_visual_link.obj; visual mesh filename=../meshes/right_thumb_proximal_visual_link.obj
- link right_thumb_touch_link: geometry collision mesh filename=../meshes/right_thumb_touch_link.obj; visual mesh filename=../meshes/right_thumb_touch_link.obj

File: src/assets/rm65/urdf/rm65.urdf (robot description, URDF)
Before this commit: robot RM65-B, 7 links, 6 joints
Links:
- link base_link: geometry collision mesh filename=../meshes/base_link.obj; visual mesh filename=../meshes/base_link.obj
- link link_1: geometry collision mesh filename=../meshes/link_1.obj; visual mesh filename=../meshes/link_1.obj
- link link_2: geometry collision mesh filename=../meshes/link_2.obj; visual mesh filename=../meshes/link_2.obj
- link link_3: geometry collision mesh filename=../meshes/link_3.obj; visual mesh filename=../meshes/link_3.obj
- link link_4: geometry collision mesh filename=../meshes/link_4.obj; visual mesh filename=../meshes/link_4.obj
- link link_5: geometry collision mesh filename=../meshes/link_5.obj; visual mesh filename=../meshes/link_5.obj
- link link_6: geometry collision mesh filename=../meshes/link_6.obj; visual mesh filename=../meshes/link_6.obj
