Commit message: Update robot asset from rm65 to rm75

File: src/assets/rm75/urdf/rm75.urdf (robot description, URDF)
Before this commit: robot RM65-B, 7 links, 6 joints
Links:
- added link link_7, mass 0.107; collision mesh filename=../meshes/link_7.obj; visual mesh filename=../meshes/link_7.obj
- link link_1: mass 1.51 -> 1.574
- link link_2: mass 1.653 -> 1.217
- link link_3: mass 0.726 -> 1.11
- link link_4: mass 0.671 -> 0.685
- link link_5: mass 0.647 -> 0.619
- link link_6: mass 0.104 -> 0.602
Joints:
- added joint joint_7: type revolute, parent link_6, child link_7, origin xyz=0 -0.144 0 rpy=1.5708 0 0, axis 0 0 1, limit lower=-6.28 upper=6.28 effort=10 velocity=3.14
- joint joint_2: origin xyz=0 0 0 rpy=1.5708 -1.5708 0 -> xyz=0 0 0 rpy=-1.5708 0 0
- joint joint_3: limit lower=-2.356 upper=2.356 effort=30 velocity=3.14 -> lower=-3.106 upper=3.106 effort=30 velocity=3.14; origin xyz=0.256 0 0 rpy=0 0 1.5708 -> xyz=0 -0.256 0 rpy=1.5708 0 0
- joint joint_4: limit lower=-3.106 upper=3.106 effort=10 velocity=3.14 -> lower=-2.356 upper=2.356 effort=30 velocity=3.14; origin xyz=0 -0.21 0 rpy=1.5708 0 0 -> xyz=0 0 0 rpy=-1.5708 0 0
- joint joint_5: limit lower=-2.234 upper=2.234 effort=10 velocity=3.14 -> lower=-3.106 upper=3.106 effort=10 velocity=3.14; origin xyz=0 0 0 rpy=-1.5708 0 0 -> xyz=0 -0.21 0 rpy=1.5708 0 0
- joint joint_6: limit lower=-6.28 upper=6.28 effort=10 velocity=3.14 -> lower=-2.234 upper=2.234 effort=10 velocity=3.14; origin xyz=0 -0.144 0 rpy=1.5708 0 0 -> xyz=0 0 0 rpy=-1.5708 0 0
